File: CNCbreakout.sch (KiCad schematic (older format))
At the start: 12 parts, among them P101 X1, P102 X2, P103 Y, P104 Z, P105 GND, P106 +24V, P107 CONN_01X02, P108 CONN_01X02, P109 CONN_01X02, P110 Z_STOP, P111 XY_STOP, P112 VFD_IN

Commit message: adjusted DE15 footprint, added aux Z-stage lines
Parts:
- added P113: Zaux1, Connect:bornier2, symbol CONN_01X02
- added P114: Zaux2, Connect:bornier2, symbol CONN_01X02
- added P115: Zaux3, Connect:bornier2, symbol CONN_01X02
Connections:
- net GND: now also P115.2 (P2)
- net SOL1: now also P113.1 (P1)
- net SOL2: now also P113.2 (P2)
- net at P110.11 (P11): now also P114.1 (P1)
- net at P110.12 (P12): now also P114.2 (P2)
- net at P110.15 (P15): now also P115.1 (P1)
Changed lines of the file:
@@
 Wire Wire Line
 	4600 4200 4750 4200
+$Comp
+L CONN_01X02 P113
+U 1 1 57FB1A8A
+P 8300 1700
+F 0 "P113" H 8300 1850 50  0000 C CNN
+F 1 "Zaux1" V 8400 1700 50  0000 C CNN
+F 2 "Connect:bornier2" H 8300 1700 50  0001 C CNN
+F 3 "" H 8300 1700 50  0000 C CNN
+	1    8300 1700
+	-1   0    0    -1
+$EndComp
+Text GLabel 8600 1650 2    60   Input ~ 0
+SOL1
+Text GLabel 8600 1750 2    60   Input ~ 0
+SOL2
+Wire Wire Line
+	8600 1750 8500 1750
+Wire Wire Line
+	8500 1650 8600 1650
+$Comp
+L CONN_01X02 P114
+U 1 1 57FB322C
+P 10900 2050
+F 0 "P114" H 10900 2200 50  0000 C CNN
+F 1 "Zaux2" V 11000 2050 50  0000 C CNN
+F 2 "Connect:bornier2" H 10900 2050 50  0001 C CNN
+F 3 "" H 10900 2050 50  0000 C CNN
+	1    10900 2050
+	1    0    0    -1
+$EndComp
+$Comp
+L CONN_01X02 P115
+U 1 1 57FB3778
+P 10900 2450
+F 0 "P115" H 10900 2600 50  0000 C CNN
+F 1 "Zaux3" V 11000 2450 50  0000 C CNN
+F 2 "Connect:bornier2" H 10900 2450 50  0001 C CNN
+F 3 "" H 10900 2450 50  0000 C CNN
+	1    10900 2450
+	1    0    0    -1
+$EndComp
+Text GLabel 10550 2650 2    60   Input ~ 0
+Z_PGND
+Wire Wire Line
+	9500 2000 10700 2000
+Wire Wire Line
+	10700 2100 9500 2100
+Wire Wire Line
+	10700 2400 9500 2400
+Wire Wire Line
+	10550 2650 10550 2500
+Wire Wire Line
+	10550 2500 10700 2500
 $EndSCHEMATC

Commit message: added thermistor
Parts:
- added P116: VFD_Speed, Connect:bornier2, symbol CONN_01X02
- added P117: VFD_Temp, Connect:bornier2, symbol CONN_01X02
- P107: value CONN_01X02 -> VFD_Stop
- P108: value CONN_01X02 -> VFD_FwdRev
- P109: value CONN_01X02 -> VFD_Aux
Connections:
- net DIn_4 is gone; now on net DIn_5: P112.8 (P8)
- net vfd_aux/GPO1 is gone; now on net DIn_1: P107.2 (P2)
- net vfd_aux/GPO2 is gone; now on net GND: P107.1 (P1)
- net vfd_aux/GPO3 is gone; now on net DIn_6: P108.2 (P2)
- net vfd_aux/GPO4 is gone; now on net DIn_3: P108.1 (P1)
- net vfd_aux/GPO5 is gone; now on net DIn_5: P109.2 (P2)
- net vfd_aux/GPO6 is gone; now on net DIn_2: P109.1 (P1)
- net DIn_5: no longer P112.4 (P4)
- net DIn_6: now also P112.4 (P4); no longer P112.9 (P9)
- net LoopA: now also P116.2 (P2)
- net LoopB: now also P116.1 (P1)
- net SpindleTherm+: now also P117.2 (P2)
- net SpindleTherm-: now also P117.1 (P1)
Other:
- note added: "VFD_PWM_DNC"
- note added: "fwd"
- note added: "rev"
- note added: "stop"
- moved on the sheet: P107, P108, P109, P113
Changed lines of the file:
@@
 $Descr A4 11693 8268
 encoding utf-8
-Sheet 1 6
+Sheet 1 5
 Title ""
 Date ""
@@
 Text GLabel 10000 4700 2    60   Input ~ 0
 DIn_3
-Text GLabel 9600 4800 2    60   Input ~ 0
+Text GLabel 10250 5200 2    60   Input ~ 0
 DIn_5
 Text GLabel 9600 5100 2    60   Input ~ 0
 DIn_2
-Text GLabel 10000 5200 2    60   Input ~ 0
-DIn_4
-Text GLabel 9600 5300 2    60   Input ~ 0
+Text GLabel 9600 4800 2    60   Input ~ 0
 DIn_6
 Text GLabel 9600 5500 2    60   Input ~ 0
@@
 Text GLabel 5150 900  2    60   Input ~ 0
 GND
-$Sheet
-S 7600 4400 900  1600
-U 5791BB59
-F0 "vfd_aux" 60
-F1 "vfd_aux.sch" 60
-F2 "GPO1" I L 7600 4600 60
-F3 "GPO2" I L 7600 4750 60
-F4 "GPO3" I L 7600 4900 60
-F5 "GPO4" I L 7600 5050 60
-F6 "GPO5" I L 7600 5200 60
-F7 "GPO6" I L 7600 5350 60
-F8 "DIN1" I R 8500 4600 60
-F9 "DIN2" I R 8500 5100 60
-F10 "DIN3" I R 8500 4700 60
-F11 "DIN4" I R 8500 5200 60
-F12 "DIN5" I R 8500 4800 60
-F13 "Din6" I R 8500 5300 60
-F14 "VFD_GND" I R 8500 5400 60
-$EndSheet
 $Sheet
 S 4900 5150 1400 750
@@
 	10500 5000 10500 4500
 Wire Wire Line
-	9500 4900 10600 4900
+	9050 4900 10600 4900
 Wire Wire Line
 	10600 4900 10600 5400
-Wire Wire Line
-	8500 5400 10700 5400
 Connection ~ 10600 5400
 Wire Wire Line
-	10000 5800 9500 5800
-Wire Wire Line
-	9600 5700 9500 5700
-Wire Wire Line
-	8500 4700 10000 4700
-Wire Wire Line
-	8500 4600 9600 4600
-Wire Wire Line
-	8500 4800 9600 4800
-Wire Wire Line
-	8500 5100 9600 5100
-Wire Wire Line
-	8500 5300 9600 5300
-Wire Wire Line
-	8500 5200 10000 5200
+	8950 5800 10000 5800
+Wire Wire Line
+	8950 5700 9600 5700
+Wire Wire Line
+	8550 4700 10000 4700
+Wire Wire Line
+	8100 4600 9600 4600
+Wire Wire Line
+	8550 4800 9600 4800
+Wire Wire Line
+	8950 5100 9600 5100
+Wire Wire Line
+	8950 5200 10250 5200
 Wire Wire Line
 	10100 5600 9500 5600
@@
 Wire Wire Line
 	2100 2400 3000 2400
-Connection ~ 9500 5400
-Connection ~ 9500 5300
 Connection ~ 9500 5200
 Connection ~ 9500 5100
@@
 L CONN_01X02 P107
 U 1 1 57B63261
-P 7150 4650
-F 0 "P107" H 7150 4800 50  0000 C CNN
-F 1 "CONN_01X02" V 7250 4650 50  0000 C CNN
-F 2 "Connect:bornier2" H 7150 4650 50  0001 C CNN
-F 3 "" H 7150 4650 50  0000 C CNN
-	1    7150 4650
-	-1   0    0    1
+P 7900 4550
+F 0 "P107" H 7900 4700 50  0000 C CNN
+F 1 "VFD_Stop" V 8000 4550 50  0000 C CNN
+F 2 "Connect:bornier2" H 7900 4550 50  0001 C CNN
+F 3 "" H 7900 4550 50  0000 C CNN
+	1    7900 4550
+	-1   0    0    -1
 $EndComp
 $Comp
 L CONN_01X02 P108
 U 1 1 57B63643
-P 7150 4950
-F 0 "P108" H 7150 5100 50  0000 C CNN
-F 1 "CONN_01X02" V 7250 4950 50  0000 C CNN
-F 2 "Connect:bornier2" H 7150 4950 50  0001 C CNN
-F 3 "" H 7150 4950 50  0000 C CNN
-	1    7150 4950
-	-1   0    0    1
+P 8350 4750
+F 0 "P108" H 8350 4900 50  0000 C CNN
+F 1 "VFD_FwdRev" V 8450 4750 50  0000 C CNN
+F 2 "Connect:bornier2" H 8350 4750 50  0001 C CNN
+F 3 "" H 8350 4750 50  0000 C CNN
+	1    8350 4750
+	-1   0    0    -1
 $EndComp
 $Comp
 L CONN_01X02 P109
 U 1 1 57B637C6
-P 7150 5250
-F 0 "P109" H 7150 5400 50  0000 C CNN
-F 1 "CONN_01X02" V 7250 5250 50  0000 C CNN
-F 2 "Connect:bornier2" H 7150 5250 50  0001 C CNN
-F 3 "" H 7150 5250 50  0000 C CNN
-	1    7150 5250
-	-1   0    0    1
-$EndComp
-Wire Wire Line
-	7350 4600 7600 4600
-Wire Wire Line
-	7600 4750 7350 4750
-Wire Wire Line
-	7350 4750 7350 4700
-Wire Wire Line
-	7350 4900 7600 4900
-Wire Wire Line
-	7600 5050 7350 5050
-Wire Wire Line
-	7350 5050 7350 5000
-Wire Wire Line
-	7350 5200 7600 5200
-Wire Wire Line
-	7600 5350 7350 5350
-Wire Wire Line
-	7350 5350 7350 5300
+P 8750 5150
+F 0 "P109" H 8750 5300 50  0000 C CNN
+F 1 "VFD_Aux" V 8850 5150 50  0000 C CNN
+F 2 "Connect:bornier2" H 8750 5150 50  0001 C CNN
+F 3 "" H 8750 5150 50  0000 C CNN
+	1    8750 5150
+	-1   0    0    -1
+$EndComp
 Wire Wire Line
 	4750 3200 4600 3200
@@
 L CONN_01X02 P113
 U 1 1 57FB1A8A
-P 8300 1700
-F 0 "P113" H 8300 1850 50  0000 C CNN
-F 1 "Zaux1" V 8400 1700 50  0000 C CNN
-F 2 "Connect:bornier2" H 8300 1700 50  0001 C CNN
-F 3 "" H 8300 1700 50  0000 C CNN
-	1    8300 1700
-	-1   0    0    -1
-$EndComp
-Text GLabel 8600 1650 2    60   Input ~ 0
+P 8400 900
+F 0 "P113" H 8400 1050 50  0000 C CNN
+F 1 "Zaux1" V 8500 900 50  0000 C CNN
+F 2 "Connect:bornier2" H 8400 900 50  0001 C CNN
+F 3 "" H 8400 900 50  0000 C CNN
+	1    8400 900
+	-1   0    0    -1
+$EndComp
+Text GLabel 8700 850  2    60   Input ~ 0
 SOL1
-Text GLabel 8600 1750 2    60   Input ~ 0
+Text GLabel 8700 950  2    60   Input ~ 0
 SOL2
 Wire Wire Line
-	8600 1750 8500 1750
-Wire Wire Line
-	8500 1650 8600 1650
+	8700 950  8600 950
+Wire Wire Line
+	8600 850  8700 850
 $Comp
 L CONN_01X02 P114
@@
 Wire Wire Line
 	10550 2500 10700 2500
+$Comp
+L CONN_01X02 P116
+U 1 1 57FB2050
+P 8750 5750
+F 0 "P116" H 8750 5900 50  0000 C CNN
+F 1 "VFD_Speed" V 8850 5750 50  0000 C CNN
+F 2 "Connect:bornier2" H 8750 5750 50  0001 C CNN
+F 3 "" H 8750 5750 50  0000 C CNN
+	1    8750 5750
+	-1   0    0    1
+$EndComp
+Text Notes 8600 4600 0    60   ~ 0
+stop
+Text Notes 8600 4700 0    60   ~ 0
+fwd
+Text Notes 8600 4800 0    60   ~ 0
+rev
+Text Notes 9550 5300 0    60   ~ 0
+VFD_PWM_DNC
+Connection ~ 9500 5700
+Connection ~ 9500 5800
+Wire Wire Line
+	8100 4500 9050 4500
+Wire Wire Line
+	9500 5400 10700 5400
+Wire Wire Line
+	9050 4500 9050 4900
+Connection ~ 9500 4900
+$Comp
+L CONN_01X02 P117
+U 1 1 57FBA8CC
+P 7600 1750
+F 0 "P117" H 7600 1900 50  0000 C CNN
+F 1 "VFD_Temp" V 7700 1750 50  0000 C CNN
+F 2 "Connect:bornier2" H 7600 1750 50  0001 C CNN
+F 3 "" H 7600 1750 50  0000 C CNN
+	1    7600 1750
+	-1   0    0    -1
+$EndComp
+Text GLabel 7900 1800 2    60   Input ~ 0
+SpindleTherm+
+Wire Wire Line
+	7900 1800 7800 1800
+Wire Wire Line
+	7800 1700 7900 1700
+Text GLabel 7900 1700 2    60   Input ~ 0
+SpindleTherm-
 $EndSCHEMATC

Commit message: added enable input connector
Parts:
- added P118: Enable, Connect:bornier2, symbol CONN_01X02
Connections:
- new net Estop_Logic/ENABLE+: P118.2 (P2)
- new net Estop_Logic/ENABLE-: P118.1 (P1)
Changed lines of the file:
@@
-$EndSheet
-$Sheet
-S 800  3900 1300 2100
-U 5791BC27
-F0 "acs_cable" 60
-F1 "acs_cable.sch" 60
-F2 "Y_GND" I R 2100 4000 60
-F3 "Y+Lim" I R 2100 4100 60
-F4 "Y-Lim" I R 2100 4200 60
-F5 "YEN+" I R 2100 4300 60
-F6 "YEN-" I R 2100 4400 60
-F7 "YHome-" I R 2100 4600 60
-F8 "Y+24V" I R 2100 4800 60
-F9 "Z_GND" I R 2100 5100 60
-F10 "Z+Lim" I R 2100 5200 60
-F11 "Z-Lim" I R 2100 5300 60
-F12 "ZEN+" I R 2100 5400 60
-F13 "ZEN-" I R 2100 5500 60
-F14 "ZHome-" I R 2100 5700 60
-F15 "Z+24V" I R 2100 5900 60
 $EndSheet
 $Sheet
@@
 F8 "X2EN+" I L 4750 3500 60
 F9 "X2EN-" I L 4750 3600 60
-F10 "ESTOP+" I R 6500 3450 60
-F11 "ESTOP-" I R 6500 3550 60
+F10 "ENABLE+" I R 6500 3350 60
+F11 "ENABLE-" I R 6500 3450 60
 $EndSheet
 Wire Wire Line
@@
 Text GLabel 7900 1700 2    60   Input ~ 0
 SpindleTherm-
+$Comp
+L CONN_01X02 P118
+U 1 1 580D988B
+P 7050 3400
+F 0 "P118" H 7050 3550 50  0000 C CNN
+F 1 "Enable" V 7150 3400 50  0000 C CNN
+F 2 "Connect:bornier2" H 7050 3400 50  0001 C CNN
+F 3 "" H 7050 3400 50  0000 C CNN
+	1    7050 3400
+	1    0    0    1
+$EndComp
+Wire Wire Line
+	6500 3350 6850 3350
+Wire Wire Line
+	6850 3450 6500 3450
+$Sheet
+S 800  3900 1300 2100
+U 5791BC27
+F0 "acs_cable" 60
+F1 "acs_cable.sch" 60
+F2 "Y_GND" I R 2100 4000 60
+F3 "Y+Lim" I R 2100 4100 60
+F4 "Y-Lim" I R 2100 4200 60
+F5 "YEN+" I R 2100 4300 60
+F6 "YEN-" I R 2100 4400 60
+F7 "YHome-" I R 2100 4600 60
+F8 "Y+24V" I R 2100 4800 60
+F9 "Z_GND" I R 2100 5100 60
+F10 "Z+Lim" I R 2100 5200 60
+F11 "Z-Lim" I R 2100 5300 60
+F12 "ZEN+" I R 2100 5400 60
+F13 "ZEN-" I R 2100 5500 60
+F14 "ZHome-" I R 2100 5700 60
+F15 "Z+24V" I R 2100 5900 60
+$EndSheet
 $EndSCHEMATC
